File: Hardware/OLED/OLED.brd (EAGLE design)
At the start: 214 x 60 mm, 16 parts, among them J2 5267-4, Q1 STP5NA50, Q2 STP5NA50, Q3 STP5NA50, SW1 EC12E_SW

Commit message: ver.1.0.5
Parts:
- removed SP1: KSS1201, buzzer:KSS1201
- added SG1: GEC-13C, buzzer:F/TMB
- moved J2 8.33 mm to (209.1, 56.4), turned to 0 degrees
- moved JP1 6.21 mm to (16.2, 19.5)
- moved JP2 6.21 mm to (54.2, 19.5)
- moved Q3 2.60 mm to (199.9, 15.5)
Connections:
- net BEEPER: now also SG1.+; no longer SP1.+
- net GND: now also SG1.-, U$1.10, U$1.7, U$1.8, U$1.9; no longer SP1.-
Routing:
- net N$9: track 52.9 -> 44.7 mm
- net SD_OUT: track 142.8 -> 149.1 mm, vias 0 -> 1
- net +12V: track 120.3 -> 126.5 mm
- net SD_CLK: track 94.7 -> 88.7 mm
- net SD_CS: track 91.2 -> 86.2 mm
- net SD_DET: track 124.7 -> 120.0 mm
- net SD_DIN: track 90.7 -> 86.1 mm
- net VCC: track 116.9 -> 114.7 mm, vias 1 -> 0
- net N$8: track 48.2 -> 46.0 mm
- net N$6: track 5.54 -> 7.57 mm
- net N$7: track 33.1 -> 34.7 mm
- net BEEPER: track 90.4 -> 89.9 mm
Other:
- board text added: "ATEAM Ventures CREATABLE D2 OLED B/D Ver. 1.1"
- board text removed: "ATEAM Ventures CREATABLE D2 OLED B/D Ver. 1.0"
