File: Hardware/OLED/OLED.sch (EAGLE design)
At the start: 16 parts, among them J2 5267-4, Q1 STP5NA50, Q2 STP5NA50, Q3 STP5NA50, SW1 EC12E_SW

Commit message: ver.1.0.5
Parts:
- removed SP1: KSS1201, buzzer:KSS1201
- added SG1: GEC-13C, buzzer:F/TMB
Connections:
- net BEEPER: now also SG1.+; no longer SP1.1
- net GND: now also SG1.-, U$1.DB0, U$1.DB1, U$1.DB2, U$1.DB3; no longer SP1.2
Changed lines of the file:
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@@
 </classes>
 <parts>
-<part name="SP1" library="buzzer" deviceset="KSS1201" device=""/>
 <part name="SW1" library="switch-alps" deviceset="EC12E_SW" device=""/>
 <part name="SUPPLY1" library="supply2" deviceset="GND" device=""/>
@@
 <part name="JP1" library="pinhead" deviceset="PINHD-2X2" device=""/>
 <part name="J2" library="con-molex-spox" deviceset="5267-4" device=""/>
+<part name="SUPPLY2" library="supply2" deviceset="GND" device=""/>
+<part name="SG1" library="buzzer" deviceset="F/TMB" device="" value="GEC-13C"/>
 </parts>
 <sheets>
@@
 </plain>
 <instances>
-<instance part="SP1" gate="1" x="137.16" y="149.86"/>
 <instance part="SW1" gate="G$1" x="50.8" y="134.62"/>
 <instance part="SW1" gate="G$2" x="66.04" y="134.62" rot="R90"/>
@@
 <instance part="JP1" gate="A" x="218.44" y="78.74"/>
 <instance part="J2" gate="G$1" x="162.56" y="114.3"/>
+<instance part="SUPPLY2" gate="GND" x="58.42" y="78.74"/>
+<instance part="SG1" gate="1" x="134.62" y="152.4" smashed="yes">
+<attribute name="NAME" x="132.08" y="158.75" size="1.778" layer="95"/>
+<attribute name="VALUE" x="139.7" y="152.4" size="1.778" layer="96"/>
+</instance>
 </instances>
 <busses>
@@
 <pinref part="SUPPLY6" gate="GND" pin="GND"/>
 <wire x1="144.78" y1="144.78" x2="144.78" y2="149.86" width="0.1524" layer="91"/>
-<pinref part="SP1" gate="1" pin="2"/>
-<wire x1="144.78" y1="149.86" x2="142.24" y2="149.86" width="0.1524" layer="91"/>
+<pinref part="SG1" gate="1" pin="-"/>
+<wire x1="139.7" y1="149.86" x2="144.78" y2="149.86" width="0.1524" layer="91"/>
 </segment>
 <segment>
@@
 <wire x1="233.68" y1="78.74" x2="233.68" y2="73.66" width="0.1524" layer="91"/>
 <pinref part="JP1" gate="A" pin="4"/>
+</segment>
+<segment>
+<pinref part="SUPPLY2" gate="GND" pin="GND"/>
+<pinref part="U$1" gate="G$1" pin="DB3"/>
+<wire x1="58.42" y1="81.28" x2="58.42" y2="83.82" width="0.1524" layer="91"/>
+<pinref part="U$1" gate="G$1" pin="DB2"/>
+<wire x1="58.42" y1="83.82" x2="58.42" y2="86.36" width="0.1524" layer="91"/>
+<wire x1="55.88" y1="86.36" x2="55.88" y2="83.82" width="0.1524" layer="91"/>
+<wire x1="55.88" y1="83.82" x2="58.42" y2="83.82" width="0.1524" layer="91"/>
+<wire x1="55.88" y1="83.82" x2="53.34" y2="83.82" width="0.1524" layer="91"/>
+<wire x1="53.34" y1="83.82" x2="50.8" y2="83.82" width="0.1524" layer="91"/>
+<pinref part="U$1" gate="G$1" pin="DB1"/>
+<wire x1="53.34" y1="86.36" x2="53.34" y2="83.82" width="0.1524" layer="91"/>
+<junction x="53.34" y="83.82"/>
+<junction x="55.88" y="83.82"/>
+<junction x="58.42" y="83.82"/>
+<pinref part="U$1" gate="G$1" pin="DB0"/>
+<wire x1="50.8" y1="83.82" x2="50.8" y2="86.36" width="0.1524" layer="91"/>
 </segment>
 </net>
@@
 <wire x1="132.08" y1="149.86" x2="111.76" y2="149.86" width="0.1524" layer="91"/>
 <label x="116.84" y="149.86" size="1.778" layer="95"/>
-<pinref part="SP1" gate="1" pin="1"/>
-</segment>
-<segment>
+<pinref part="SG1" gate="1" pin="+"/>
+</segment>
+<segment>
